Commit message: rviz gazebo match back

File: src/arpa_description/urdf/arpa_system.urdf.xacro (robot description, xacro)
@@ -90,3 +90,12 @@
       </gazebo>
     </xacro:if>
+    <!-- Add linear actuator joint to ros2_control for Gazebo simulation -->
+    <xacro:if value="$(arg sim_gazebo)">
+      <ros2_control name="LinearActuatorSystem" type="system">
+        <hardware>
+          <plugin>gazebo_ros2_control/GazeboSystem</plugin>
+        </hardware>
+        <xacro:linear_actuator_ros2_control/>
+      </ros2_control>
+    </xacro:if>
 </robot>

File: src/arpa_description/urdf/arpa_system_macro.urdf.xacro (robot description, xacro)
@@ -4,4 +4,5 @@
   <xacro:include filename="$(find arpa_description)/urdf/gantry.xacro"/>
   <xacro:include filename="$(find arpa_description)/urdf/linear_actuator.xacro"/>
+  <xacro:include filename="$(find arpa_description)/urdf/linear_actuator_ros2_control.xacro"/>
   <xacro:include filename="$(find arpa_description)/urdf/tool_holder.xacro"/>
   <xacro:include filename="$(find ur_description)/urdf/ur_macro.xacro"/>

File: src/arpa_description/urdf/linear_actuator.xacro (robot description, xacro)
@@ -48,6 +48,6 @@
       </inertial>
     </link>
-    <!-- Fixed joints (pillars attach to beam) -->
-    <!-- <joint name="linear_actuator_to_linear_actuator_plate_joint" type="prismatic">
+    <!-- Prismatic joint for linear actuator movement -->
+    <joint name="linear_actuator_to_linear_actuator_plate_joint" type="prismatic">
       <parent link="linear_actuator_link"/>
       <child link="linear_actuator_plate_link"/>
@@ -55,10 +55,4 @@
       <axis xyz="1 0 0"/>
       <limit lower="-1.845" upper="0.0" effort="100.0" velocity="0.5"/>
-    </joint> -->
-    <joint name="linear_actuator_to_linear_actuator_plate_joint" type="fixed">
-      <parent link="linear_actuator_link"/>
-      <child link="linear_actuator_plate_link"/>
-      <!-- <origin xyz="1.0244 0 -0.04375" rpy="0 0 0"/> -->
-      <origin xyz="0.3556 0 -0.04375" rpy="0 0 0"/>
     </joint>
   </xacro:macro>
