Commit message: trying to get linear actuator in the loop

File: src/arpa_description/urdf/arpa_system.urdf.xacro (robot description, xacro)
@@ -10,5 +10,5 @@
     <!-- parameters -->
     <xacro:arg name="tf_prefix" default="" />
-    <xacro:arg name="joint_limit_params" default="$(find ur_description)/config/$(arg ur_type)/joint_limits.yaml"/>
+    <xacro:arg name="joint_limit_params" default="$(find arpa_description)/config/joint_limits.yaml"/>
     <xacro:arg name="kinematics_params" default="$(find ur_description)/config/$(arg ur_type)/default_kinematics.yaml"/>
     <xacro:arg name="physical_params" default="$(find ur_description)/config/$(arg ur_type)/physical_parameters.yaml"/>
@@ -98,4 +98,10 @@
         </plugin>
       </gazebo>
+      <ros2_control name="LinearActuatorSystem" type="system">
+        <hardware>
+          <plugin>gazebo_ros2_control/GazeboSystem</plugin>
+        </hardware>
+        <xacro:linear_actuator_ros2_control/>
+      </ros2_control>
     </xacro:if>
 </robot>

File: src/arpa_description/urdf/arpa_system_macro.urdf.xacro (robot description, xacro)
@@ -4,4 +4,5 @@
   <xacro:include filename="$(find arpa_description)/urdf/gantry.xacro"/>
   <xacro:include filename="$(find arpa_description)/urdf/linear_actuator.xacro"/>
+  <xacro:include filename="$(find arpa_description)/urdf/linear_actuator_ros2_control.xacro"/>
   <xacro:include filename="$(find arpa_description)/urdf/tool_holder.xacro"/>
   <xacro:include filename="$(find ur_description)/urdf/ur_macro.xacro"/>

File: src/arpa_moveit_config/srdf/arpa_system_macro.srdf.xacro (robot description, xacro)
@@ -2,4 +2,7 @@
 <robot xmlns:xacro="http://wiki.ros.org/xacro">
   <xacro:macro name="arpa_system" params="name prefix">
+    <group name="linear_actuator_axis">
+      <joint name="linear_actuator_to_linear_actuator_plate_joint"/>
+    </group>
     <group name="${prefix}${name}ur_manipulator">
       <chain base_link="${prefix}base_link" tip_link="${prefix}tool0"/>
@@ -15,4 +18,34 @@
       <joint name="wrist_2_joint" value="0"/>
       <joint name="wrist_3_joint" value="0"/>
+    </group_state>
+    <group name="ur16e_on_gantry">
+      <!-- Explicit joint listing ensures all 7 DOF are explored during planning -->
+      <joint name="linear_actuator_to_linear_actuator_plate_joint"/>
+      <joint name="shoulder_pan_joint"/>
+      <joint name="shoulder_lift_joint"/>
+      <joint name="elbow_joint"/>
+      <joint name="wrist_1_joint"/>
+      <joint name="wrist_2_joint"/>
+      <joint name="wrist_3_joint"/>
+    </group>
+    <group_state name="actuator_home" group="linear_actuator_axis">
+      <joint name="linear_actuator_to_linear_actuator_plate_joint" value="-1.12"/>
+    </group_state>
+    <group_state name="arm_home" group="ur_manipulator">
+      <joint name="elbow_joint" value="2.3387"/>
+      <joint name="shoulder_lift_joint" value="-2.6179"/>
+      <joint name="shoulder_pan_joint" value="-2.7576"/>
+      <joint name="wrist_1_joint" value="-1.29154"/>
+      <joint name="wrist_2_joint" value="-4.6949"/>
+      <joint name="wrist_3_joint" value="1.1868"/>
+    </group_state>
+    <group_state name="arpa_home" group="ur16e_on_gantry">
+      <joint name="linear_actuator_to_linear_actuator_plate_joint" value="-1.12"/>
+      <joint name="shoulder_pan_joint" value="-2.7576"/>
+      <joint name="shoulder_lift_joint" value="-2.6179"/>
+      <joint name="elbow_joint" value="2.3386"/>
+      <joint name="wrist_1_joint" value="-1.2915"/>
+      <joint name="wrist_2_joint" value="-4.6948"/>
+      <joint name="wrist_3_joint" value="1.1868"/>
     </group_state>
     <end_effector name="end_effector_and_tool" parent_link="${prefix}tool0" group="${prefix}end_effector" parent_group="${prefix}ur_manipulator"/>
@@ -38,6 +71,5 @@
     <disable_collisions link1="${prefix}base_link_inertia" link2="${prefix}wrist_1_link" reason="Never"/>
     <disable_collisions link1="${prefix}forearm_link" link2="${prefix}left_leg_link" reason="Never"/>
-    <disable_collisions link1="${prefix}forearm_link" link2="${prefix}pillar_left_link" reason="Never"/>
-    <disable_collisions link1="${prefix}forearm_link" link2="${prefix}pillar_right_link" reason="Never"/>
+    <disable_collisions link1="${prefix}forearm_link" link2="${prefix}pillar_left_link" reason="Default"/>
     <disable_collisions link1="${prefix}forearm_link" link2="${prefix}right_leg_link" reason="Never"/>
     <disable_collisions link1="${prefix}forearm_link" link2="${prefix}upper_arm_link" reason="Adjacent"/>
@@ -75,17 +107,7 @@
     <disable_collisions link1="${prefix}pillar_left_link" link2="${prefix}right_leg_link" reason="Never"/>
     <disable_collisions link1="${prefix}pillar_left_link" link2="${prefix}shoulder_link" reason="Never"/>
-    <disable_collisions link1="${prefix}pillar_left_link" link2="${prefix}upper_arm_link" reason="Never"/>
-    <disable_collisions link1="${prefix}pillar_left_link" link2="${prefix}wrist_1_link" reason="Never"/>
-    <disable_collisions link1="${prefix}pillar_left_link" link2="${prefix}wrist_2_link" reason="Never"/>
-    <disable_collisions link1="${prefix}pillar_left_link" link2="${prefix}wrist_3_link" reason="Never"/>
     <disable_collisions link1="${prefix}pillar_right_link" link2="${prefix}right_leg_link" reason="Adjacent"/>
     <disable_collisions link1="${prefix}pillar_right_link" link2="${prefix}shoulder_link" reason="Never"/>
-    <disable_collisions link1="${prefix}pillar_right_link" link2="${prefix}tool_center_link" reason="Never"/>
-    <disable_collisions link1="${prefix}pillar_right_link" link2="${prefix}tool_head_link" reason="Never"/>
-    <disable_collisions link1="${prefix}pillar_right_link" link2="${prefix}tool_holder_link" reason="Never"/>
     <disable_collisions link1="${prefix}pillar_right_link" link2="${prefix}upper_arm_link" reason="Never"/>
-    <disable_collisions link1="${prefix}pillar_right_link" link2="${prefix}wrist_1_link" reason="Never"/>
-    <disable_collisions link1="${prefix}pillar_right_link" link2="${prefix}wrist_2_link" reason="Never"/>
-    <disable_collisions link1="${prefix}pillar_right_link" link2="${prefix}wrist_3_link" reason="Never"/>
     <disable_collisions link1="${prefix}right_leg_link" link2="${prefix}shoulder_link" reason="Never"/>
     <disable_collisions link1="${prefix}right_leg_link" link2="${prefix}tool_center_link" reason="Never"/>

Commit message: working simulation with arpa_system.ros2_controllers.xacro

File: src/arpa_description/urdf/arpa_system.urdf.xacro (robot description, xacro)
@@ -44,5 +44,5 @@
     <xacro:arg name="sim_gazebo" default="false" />
     <xacro:arg name="sim_ignition" default="false" />
-    <xacro:arg name="simulation_controllers" default="" />
+    <!-- <xacro:arg name="simulation_controllers" default="" /> -->
     <!-- initial position for simulations (Fake Hardware, Gazebo, Ignition) -->
     <xacro:arg name="initial_positions_file" default="$(find ur_description)/config/initial_positions.yaml"/>
@@ -65,4 +65,5 @@
         safety_k_position="$(arg safety_k_position)"
         use_fake_hardware="$(arg use_fake_hardware)"
+        generate_ros2_control_tag="false"
         fake_sensor_commands="$(arg fake_sensor_commands)"
         sim_gazebo="$(arg sim_gazebo)"

File: src/arpa_description/urdf/arpa_system_macro.urdf.xacro (robot description, xacro)
@@ -7,30 +7,7 @@
   <xacro:include filename="$(find arpa_description)/urdf/tool_holder.xacro"/>
   <xacro:include filename="$(find ur_description)/urdf/ur_macro.xacro"/>
+  <xacro:include filename="$(find arpa_moveit_config)/config/arpa_system.ros2_control.xacro" />
   <xacro:include filename="$(find parker_controller_interface)/urdf/parker_linear_actuator.ros2_control.xacro" />
-  <!-- <xacro:arg name="tf_prefix" default="" />
-  <xacro:arg name="joint_limit_params" default="$(find ur_description)/config/$(arg ur_type)/joint_limits.yaml"/>
-  <xacro:arg name="kinematics_params" default="$(find ur_description)/config/$(arg ur_type)/default_kinematics.yaml"/>
-  <xacro:arg name="physical_params" default="$(find ur_description)/config/$(arg ur_type)/physical_parameters.yaml"/>
-  <xacro:arg name="visual_params" default="$(find ur_description)/config/$(arg ur_type)/visual_parameters.yaml"/>
-  <xacro:arg name="transmission_hw_interface" default=""/>
-  <xacro:arg name="safety_limits" default="false"/>
-  <xacro:arg name="safety_pos_margin" default="0.15"/>
-  <xacro:arg name="safety_k_position" default="20"/>
-  <xacro:arg name="mock_sensor_commands" default="false" /> -->
-  <!--When using gazebo simulations absolute paths are necessary.-->
-  <!-- <xacro:arg name="force_abs_paths" default="false" /> -->
-  <!-- initial position for simulations (Mock Hardware, Gazebo, Ignition) -->
-  <!-- <xacro:arg name="initial_positions_file" default="$(find ur_description)/config/initial_positions.yaml"/> -->
-  <!-- convert to property to use substitution in function -->
-  <!-- <xacro:property name="initial_positions_file" default="$(arg initial_positions_file)"/> -->
-  <!--
-    ARPA system macro
-    Exposes UR parameters so your wrapper/launch can pass:
-      - robot_ip
-      - script/recipes (indirectly via generate_ros2_control_tag path)
-      - use_fake_hardware
-      - safety settings
-      - *and* which UR model config files to use
-  -->
+  <!-- Macro definition -->
   <xacro:macro name="arpa_system_macro" params="
     name
@@ -42,5 +19,5 @@
     physical_parameters_file
     visual_parameters_file
-    generate_ros2_control_tag:=true
+    generate_ros2_control_tag:=false
     transmission_hw_interface:=hardware_interface/PositionJointInterface
     safety_limits:=false
@@ -84,5 +61,4 @@
       <origin xyz="0 0 1.9419" rpy="0 0 0"/>
     </joint>
-    <xacro:linear_actuator/>
     <!-- Fixed transform from gantry_link to linear_actuator_link -->
     <joint name="gantry_to_linear_actuator" type="fixed">
@@ -91,4 +67,5 @@
       <origin xyz="0 0 -0.11375" rpy="0 0 0"/>
     </joint>
+    <xacro:linear_actuator/>
     <link name="arm_mount_plate">
       <visual>
@@ -138,4 +115,5 @@
         visual_parameters_file="${visual_parameters_file}"
         transmission_hw_interface="${transmission_hw_interface}"
+        generate_ros2_control_tag="false"
         safety_limits="${safety_limits}"
         safety_pos_margin="${safety_pos_margin}"
@@ -170,23 +148,43 @@
     <!-- Tool holder on tool0 -->
     <xacro:tool_holder parent_link="tool0"/>
-    <!-- Gazebo Classic plugins for simulation -->
-    <xacro:if value="$(arg sim_gazebo)">
+    <!-- ros2_control tag for the whole system -->
+    <xacro:arpa_system_ros2_control
+        name="${name}"
+        tf_prefix="${tf_prefix}"
+        use_fake_hardware="${use_fake_hardware}"
+        fake_sensor_commands="${fake_sensor_commands}"
+        sim_gazebo="${sim_gazebo}"
+        sim_ignition="${sim_ignition}"
+        headless_mode="${headless_mode}"
+        initial_positions="${xacro.load_yaml(initial_positions_file)}"
+        use_tool_communication="${use_tool_communication}"
+        tool_voltage="${tool_voltage}"
+        tool_parity="${tool_parity}"
+        tool_baud_rate="${tool_baud_rate}"
+        tool_stop_bits="${tool_stop_bits}"
+        tool_rx_idle_chars="${tool_rx_idle_chars}"
+        tool_tx_idle_chars="${tool_tx_idle_chars}"
+        tool_device_name="${tool_device_name}"
+        tool_tcp_port="${tool_tcp_port}"
+        robot_ip="${robot_ip}"
+        script_filename="${script_filename}"
+        output_recipe_filename="${output_recipe_filename}"
+        input_recipe_filename="${input_recipe_filename}"
+        reverse_ip="${reverse_ip}"
+        script_command_port="${script_command_port}"
+        reverse_port="${reverse_port}"
+        script_sender_port="${script_sender_port}"
+        trajectory_port="${trajectory_port}"
+    />
+    <!-- Gazebo ros2_control plugin - required for controller_manager in simulation -->
+    <xacro:if value="${sim_gazebo}">
       <gazebo>
         <plugin filename="libgazebo_ros2_control.so" name="gazebo_ros2_control">
-          <parameters>$(arg simulation_controllers)</parameters>
+          <robot_param>robot_description</robot_param>
+          <robot_param_node>robot_state_publisher</robot_param_node>
+          <parameters>$(find arpa_moveit_config)/config/arpa_controllers.yaml</parameters>
         </plugin>
       </gazebo>
-      <ros2_control name="LinearActuatorSystem" type="system">
-        <hardware>
-          <plugin>gazebo_ros2_control/GazeboSystem</plugin>
-        </hardware>
-        <xacro:linear_actuator_ros2_control/>
-      </ros2_control>
     </xacro:if>
-    <!-- Add ros2_control hardware interface -->
-    <!-- <xacro:parker_linear_actuator_ros2_control
-      name="ParkerControllerInterface"
-      host="192.168.100.1"
-      port="5002"/> -->
   </xacro:macro>
 </robot>

File: src/arpa_moveit_config/config/arpa_system.ros2_control.xacro (robot description, xacro)
@@ -10,6 +10,5 @@
     use_tool_communication:=false
     script_filename output_recipe_filename
-    input_recipe_filename tf_prefix
-    hash_kinematics robot_ip
+    input_recipe_filename tf_prefix robot_ip
     tool_voltage:=0 tool_parity:=0 tool_baud_rate:=115200 tool_stop_bits:=1
     tool_rx_idle_chars:=1.5 tool_tx_idle_chars:=3.5 tool_device_name:=/tmp/ttyUR tool_tcp_port:=54321
@@ -53,5 +52,4 @@
           <param name="servoj_lookahead_time">0.03</param>
           <param name="use_tool_communication">${use_tool_communication}</param>
-          <param name="kinematics/hash">${hash_kinematics}</param>
           <param name="tool_voltage">${tool_voltage}</param>
           <param name="tool_parity">${tool_parity}</param>
@@ -143,4 +141,15 @@
         <state_interface name="effort"/>
       </joint>
+      <!-- Linear actuator joint for simulation -->
+      <xacro:if value="${sim_gazebo or sim_ignition}">
+        <joint name="linear_actuator_to_linear_actuator_plate_joint">
+          <command_interface name="position"/>
+          <command_interface name="velocity"/>
+          <state_interface name="position">
+            <param name="initial_value">0.0</param>
+          </state_interface>
+          <state_interface name="velocity"/>
+        </joint>
+      </xacro:if>
       <xacro:unless value="${sim_gazebo or sim_ignition}">
         <sensor name="${tf_prefix}tcp_fts_sensor">
