Commit message: battery scan works

File: src/arpa_description/urdf/linear_actuator.xacro (robot description, xacro)
@@ -55,5 +55,5 @@
       <origin xyz="1.0244 0 -0.04375" rpy="0 0 0"/>
       <axis xyz="-1 0 0"/>
-      <limit lower="0.1" upper="2.0" effort="100.0" velocity="0.5"/>
+      <limit lower="0.25" upper="1.75" effort="100.0" velocity="0.5"/>
     </joint>
   </xacro:macro>
