Commit message: begining real experiments with moveit

File: src/arpa_description/urdf/tool_holder.xacro (robot description, xacro)
@@ -77,5 +77,6 @@
       <collision>
         <geometry>
-          <cylinder radius=".01" length="0.12"/>
+          <!-- <cylinder radius=".01" length="0.12"/> -->
+          <cylinder radius=".01" length="0.29"/>
         </geometry>
       </collision>
@@ -88,5 +89,6 @@
       <parent link="tool_center_link"/>
       <child link="tool_head_link"/>
-      <origin xyz="0.06 0 0.175" rpy="0 ${pi/2.} 0"/>
+      <!-- <origin xyz="0.06 0 0.175" rpy="0 ${pi/2.} 0"/> -->
+      <origin xyz="0.145 0 0.175" rpy="0 ${pi/2.} 0"/>
     </joint>
   </xacro:macro>

Commit message: attempted tool fix needs work, solved delay problem on ur_control ros2 stuff

File: src/arpa_description/urdf/tool_holder.xacro (robot description, xacro)
@@ -77,6 +77,6 @@
       <collision>
         <geometry>
-          <!-- <cylinder radius=".01" length="0.12"/> -->
-          <cylinder radius=".01" length="0.29"/>
+          <cylinder radius=".01" length="0.12"/>
+          <!-- <cylinder radius=".01" length="0.29"/> -->
         </geometry>
       </collision>
@@ -89,6 +89,6 @@
       <parent link="tool_center_link"/>
       <child link="tool_head_link"/>
-      <!-- <origin xyz="0.06 0 0.175" rpy="0 ${pi/2.} 0"/> -->
-      <origin xyz="0.145 0 0.175" rpy="0 ${pi/2.} 0"/>
+      <origin xyz="0.06 0 0.175" rpy="0 ${pi/2.} 0"/>
+      <!-- <origin xyz="0.145 0 0.175" rpy="0 ${pi/2.} 0"/> -->
     </joint>
   </xacro:macro>

Commit message: update urdf

File: src/arpa_description/urdf/tool_holder.xacro (robot description, xacro)
@@ -70,5 +70,5 @@
       <visual>
         <geometry>
-          <cylinder radius=".005" length="0.1"/>
+          <cylinder radius=".01" length="0.18"/>
         </geometry>
         <origin xyz="0 0 0"/>
@@ -77,6 +77,6 @@
       <collision>
         <geometry>
-          <cylinder radius=".01" length="0.12"/>
-          <!-- <cylinder radius=".01" length="0.29"/> -->
+          <!-- <cylinder radius=".01" length="0.12"/> -->
+          <cylinder radius=".01" length="0.18"/>
         </geometry>
       </collision>
@@ -89,6 +89,6 @@
       <parent link="tool_center_link"/>
       <child link="tool_head_link"/>
-      <origin xyz="0.06 0 0.175" rpy="0 ${pi/2.} 0"/>
-      <!-- <origin xyz="0.145 0 0.175" rpy="0 ${pi/2.} 0"/> -->
+      <!-- <origin xyz="0.06 0 0.175" rpy="0 ${pi/2.} 0"/> -->
+      <origin xyz="0.09 0 0.175" rpy="0 ${pi/2.} 0"/>
     </joint>
   </xacro:macro>

File: src/arpa_moveit_config/srdf/arpa_system_macro.srdf.xacro (robot description, xacro)
@@ -104,4 +104,7 @@
     <disable_collisions link1="${prefix}linear_actuator_plate_link" link2="${prefix}right_leg_link" reason="Never"/>
     <disable_collisions link1="${prefix}linear_actuator_plate_link" link2="${prefix}shoulder_link" reason="Never"/>
+    <disable_collisions link1="${prefix}linear_actuator_link" link2="${prefix}linear_actuator_plate_link" reason="Adjacent"/>
+    <disable_collisions link1="${prefix}linear_actuator_link" link2="${prefix}actuator_motor_link" reason="Adjacent"/>
+    <disable_collisions link1="${prefix}linear_actuator_plate_link" link2="${prefix}actuator_motor_link" reason="Adjacent"/>
     <disable_collisions link1="${prefix}pillar_left_link" link2="${prefix}pillar_right_link" reason="Never"/>
     <disable_collisions link1="${prefix}pillar_left_link" link2="${prefix}right_leg_link" reason="Never"/>

File: src/parker_controller_interface/srdf/parker_linear_actuator_macro.srdf.xacro (robot description, xacro)
@@ -10,4 +10,6 @@
     <virtual_joint name="world" type="fixed" parent_frame="world" child_link="${prefix}floor_link"/>
     <disable_collisions link1="${prefix}linear_actuator_link" link2="${prefix}linear_actuator_plate_link" reason="Adjacent"/>
+    <disable_collisions link1="${prefix}linear_actuator_link" link2="${prefix}actuator_motor_link" reason="Adjacent"/>
+    <disable_collisions link1="${prefix}linear_actuator_plate_link" link2="${prefix}actuator_motor_link" reason="Adjacent"/>
   </xacro:macro>
 </robot>

File: src/parker_controller_interface/urdf/parker_linear_actuator_macro.urdf.xacro (robot description, xacro)
@@ -32,4 +32,30 @@
       <child link="linear_actuator_link"/>
       <origin xyz="${origin.split(' ')[0]} ${origin.split(' ')[1]} ${origin.split(' ')[2]}" rpy="${origin.split(' ')[3]} ${origin.split(' ')[4]} ${origin.split(' ')[5]}"/>
+    </joint>
+    <link name="actuator_motor_link">
+      <visual>
+        <geometry>
+          <box size="0.095 0.335 0.095"/>
+        </geometry>
+        <origin xyz="0 0 0"/>
+        <material name="actuator_gray">
+          <color rgba="0.75 0.75 0.75 1"/>
+        </material>
+      </visual>
+      <collision>
+        <geometry>
+          <box size="0.095 0.335 0.095"/>
+        </geometry>
+      </collision>
+      <inertial>
+        <mass value="5.0"/>
+        <inertia ixx="0.01" iyy="0.01" izz="0.01" ixy="0" ixz="0" iyz="0"/>
+      </inertial>
+    </link>
+    <!-- Fixed joint for actuator motor -->
+    <joint name="linear_actuator_to_actuator_motor_joint" type="fixed">
+      <parent link="linear_actuator_link"/>
+      <child link="actuator_motor_link"/>
+      <origin xyz="1.245 -0.2425 0.0" rpy="0 0 0"/>
     </joint>
     <link name="linear_actuator_plate_link">

Commit message: add TSP and cost matrix computation, simplify end effector collision object as a box

File: src/arpa_description/urdf/tool_holder.xacro (robot description, xacro)
@@ -26,7 +26,7 @@
       <collision>
         <geometry>
-          <mesh filename="file://${mesh_filename}" scale="${scale}"/>
+          <box size="0.365 0.125 0.105"/>
         </geometry>
-        <origin xyz="${origin_xyz}" rpy="${origin_rpy}"/>
+        <origin xyz="0.055 -0.006 0.015" rpy="${origin_rpy}"/>
       </collision>
       <inertial>

Commit message: working on fixing the battery scan planning problem

File: src/arpa_description/urdf/tool_holder.xacro (robot description, xacro)
@@ -8,5 +8,6 @@
   <xacro:macro name="tool_holder" params="
       parent_link
-      mesh_filename:='$(find arpa_description)/meshes/tool_holder_v2.stl'
+      visual_mesh_filename:='$(find arpa_description)/meshes/tool_holder_v2_visual.stl'
+      collision_mesh_filename:='$(find arpa_description)/meshes/tool_holder_v2_collision.stl'
       mass:=0.5
       origin_xyz:='-0.0055 -0.0055 -.006'
@@ -17,5 +18,5 @@
       <visual>
         <geometry>
-          <mesh filename="file://${mesh_filename}" scale="${scale}"/>
+          <mesh filename="file://${visual_mesh_filename}" scale="${scale}"/>
         </geometry>
         <origin xyz="${origin_xyz}" rpy="${origin_rpy}"/>
@@ -26,7 +27,7 @@
       <collision>
         <geometry>
-          <box size="0.365 0.125 0.105"/>
+          <mesh filename="file://${collision_mesh_filename}" scale="${scale}"/>
         </geometry>
-        <origin xyz="0.055 -0.006 0.015" rpy="${origin_rpy}"/>
+        <origin xyz="${origin_xyz}" rpy="${origin_rpy}"/>
       </collision>
       <inertial>
@@ -44,22 +45,5 @@
       <origin xyz="${origin_xyz}" rpy="${origin_rpy}"/>
     </joint>
-    <link name="tool_center_link">
-      <visual>
-        <geometry>
-          <cylinder radius=".025" length="0.4"/>
-        </geometry>
-        <origin xyz="0 0 0"/>
-        <material name="gantry_gray"/>
-      </visual>
-      <collision>
-        <geometry>
-          <cylinder radius=".025" length="0.4"/>
-        </geometry>
-      </collision>
-      <inertial>
-        <mass value="5.0"/>
-        <inertia ixx="0.01" iyy="0.01" izz="0.01" ixy="0" ixz="0" iyz="0"/>
-      </inertial>
-    </link>
+    <link name="tool_center_link"/>
     <joint name="mount_to_center_joint" type="fixed">
       <parent link="tool_holder_link"/>

File: src/arpa_moveit_config/srdf/arpa_system_macro.srdf.xacro (robot description, xacro)
@@ -3,4 +3,7 @@
   <xacro:macro name="arpa_system" params="name prefix">
     <!-- ur_manipulator first so Motion Planning plugin defaults to arm-only group -->
+    <!-- <group name="ur16e_on_gantry">
+      <chain base_link="linear_actuator_plate_link" tip_link="tool0"/>
+    </group> -->
     <group name="${prefix}${name}ur_manipulator">
       <chain base_link="${prefix}base_link" tip_link="${prefix}tool0"/>
@@ -10,5 +13,5 @@
     </group>
     <group name="${prefix}end_effector">
-      <chain base_link="${prefix}tool0" tip_link="${prefix}tool_head_link"/>
+      <chain base_link="${prefix}wrist_3_joint" tip_link="${prefix}tool_head_link"/>
     </group>
     <group_state group="ur_manipulator" name="home">
@@ -21,5 +24,4 @@
     </group_state>
     <group name="ur16e_on_gantry">
-      <!-- Explicit joint listing ensures all 7 DOF are explored during planning -->
       <joint name="linear_actuator_to_linear_actuator_plate_joint"/>
       <joint name="shoulder_pan_joint"/>

Commit message: screw removal from vision + LA planning + triangle area cost

File: src/arpa_description/urdf/tool_holder.xacro (robot description, xacro)
@@ -24,9 +24,15 @@
         </material>
       </visual>
-      <collision>
+      <!-- <collision>
         <geometry>
           <box size="0.365 0.125 0.105"/>
         </geometry>
         <origin xyz="0.055 -0.006 0.015" rpy="${origin_rpy}"/>
+      </collision> -->
+      <collision>
+        <geometry>
+          <mesh filename="file://${mesh_filename}" scale="${scale}"/>
+        </geometry>
+        <origin xyz="${origin_xyz}" rpy="${origin_rpy}"/>
       </collision>
       <inertial>
@@ -96,5 +102,5 @@
       <parent link="ratchet_extension_link"/>
       <child link="tool_head_link"/>
-      <origin xyz="0.0 0 0.09" rpy="0 0 0"/>
+      <origin xyz="0.0 0 0.09" rpy="0 0 -${pi/2.}"/>
     </joint>
   </xacro:macro>

Commit message: simplify motion control node, removal from vision up to date, update submodules

File: src/arpa_description/urdf/tool_holder.xacro (robot description, xacro)
@@ -72,4 +72,5 @@
       <child link="tool_center_link"/>
       <origin xyz="0.0575 0 -0.03" rpy="0 0 0"/>
+      <!-- <origin xyz="0.0575 -0.005 0.0"  rpy="0 0 0"/> -->
     </joint>
     <link name="ratchet_extension_link">
