Commit message: redoing moveit setup assistant and the launch files for sim

File: src/arpa_description/urdf/arpa_system_macro.urdf.xacro (robot description, xacro)
@@ -32,33 +32,44 @@
   -->
   <xacro:macro name="arpa_system_macro" params="
-      ur_name:=''
-      tf_prefix:=''
-      sim_gazebo:=false
-      sim_ignition:=false
-      robot_ip:=''
-      reverse_ip:='0.0.0.0'
-      joint_limits_parameters_file:=''
-      kinematics_parameters_file:=''
-      physical_parameters_file:=''
-      visual_parameters_file:=''
-      script_filename:='to_be_filled_by_ur_robot_driver'
-      input_recipe_filename:='to_be_filled_by_ur_robot_driver'
-      output_recipe_filename:='to_be_filled_by_ur_robot_driver'
-      generate_ros2_control_tag:=true
-      transmission_hw_interface:='hardware_interface/PositionJointInterface'
-      use_fake_hardware:=false
-      fake_sensor_commands:=false
-      safety_limits:=false
-      safety_pos_margin:=0.15
-      safety_k_position:=20
-      headless_mode:=false
-      use_tool_communication:=false
-      tool_voltage:=0
-      tool_parity:=0
-      tool_baud_rate:=115200
-      tool_stop_bits:=1
-      tool_rx_idle_chars:=1.5
-      tool_tx_idle_chars:=3.5
-    ">
+    name
+    tf_prefix
+    parent
+    *origin
+    joint_limits_parameters_file
+    kinematics_parameters_file
+    physical_parameters_file
+    visual_parameters_file
+    generate_ros2_control_tag:=true
+    transmission_hw_interface:=hardware_interface/PositionJointInterface
+    safety_limits:=false
+    safety_pos_margin:=0.15
+    safety_k_position:=20
+    use_fake_hardware:=false
+    fake_sensor_commands:=false
+    sim_gazebo:=false
+    sim_ignition:=false
+    headless_mode:=false
+    initial_positions:=${dict(shoulder_pan_joint=0.0,shoulder_lift_joint=-1.57,elbow_joint=0.0,wrist_1_joint=-1.57,wrist_2_joint=0.0,wrist_3_joint=0.0)}
+    use_tool_communication:=false
+    tool_voltage:=0
+    tool_parity:=0
+    tool_baud_rate:=115200
+    tool_stop_bits:=1
+    tool_rx_idle_chars:=1.5
+    tool_tx_idle_chars:=3.5
+    tool_device_name:=/tmp/ttyUR
+    tool_tcp_port:=54321
+    robot_ip:=0.0.0.0
+    script_filename:=to_be_filled_by_ur_robot_driver
+    output_recipe_filename:=to_be_filled_by_ur_robot_driver
+    input_recipe_filename:=to_be_filled_by_ur_robot_driver
+    reverse_port:=50001
+    script_sender_port:=50002
+    reverse_ip:=0.0.0.0
+    script_command_port:=50004
+    trajectory_port:=50003
+    non_blocking_read:=true
+    keep_alive_count:=2"
+    >
     <!-- Map link -->
     <link name="floor_link"/>
@@ -117,52 +128,42 @@
     <!-- UR robot -->
     <xacro:ur_robot
-      name="${ur_name}"
-      tf_prefix="${tf_prefix}"
-      parent="ur_base_link"
-      joint_limits_parameters_file="${joint_limits_parameters_file}"
-      kinematics_parameters_file="${kinematics_parameters_file}"
-      physical_parameters_file="${physical_parameters_file}"
-      visual_parameters_file="${visual_parameters_file}"
-      script_filename="${script_filename}"
-      input_recipe_filename="${input_recipe_filename}"
-      output_recipe_filename="${output_recipe_filename}"
-      generate_ros2_control_tag="${generate_ros2_control_tag}"
-      transmission_hw_interface="${transmission_hw_interface}"
-      use_fake_hardware="${use_fake_hardware}"
-      fake_sensor_commands="${fake_sensor_commands}"
-      safety_limits="${safety_limits}"
-      safety_pos_margin="${safety_pos_margin}"
-      safety_k_position="${safety_k_position}"
-      sim_gazebo="${sim_gazebo}"
-      sim_ignition="${sim_ignition}"
-      headless_mode="${headless_mode}"
-      use_tool_communication="${use_tool_communication}"
-      tool_voltage="${tool_voltage}"
-      tool_parity="${tool_parity}"
-      tool_baud_rate="${tool_baud_rate}"
-      tool_stop_bits="${tool_stop_bits}"
-      tool_rx_idle_chars="${tool_rx_idle_chars}"
-      tool_tx_idle_chars="${tool_tx_idle_chars}"
-      robot_ip="${robot_ip}"
-      reverse_ip="${reverse_ip}"
+        name="${name}"
+        tf_prefix="${tf_prefix}"
+        parent="ur_base_link"
+        joint_limits_parameters_file="${joint_limits_parameters_file}"
+        kinematics_parameters_file="${kinematics_parameters_file}"
+        physical_parameters_file="${physical_parameters_file}"
+        visual_parameters_file="${visual_parameters_file}"
+        transmission_hw_interface="${transmission_hw_interface}"
+        safety_limits="${safety_limits}"
+        safety_pos_margin="${safety_pos_margin}"
+        safety_k_position="${safety_k_position}"
+        use_fake_hardware="${use_fake_hardware}"
+        fake_sensor_commands="${fake_sensor_commands}"
+        sim_gazebo="${sim_gazebo}"
+        sim_ignition="${sim_ignition}"
+        headless_mode="${headless_mode}"
+        initial_positions="${xacro.load_yaml(initial_positions_file)}"
+        use_tool_communication="${use_tool_communication}"
+        tool_voltage="${tool_voltage}"
+        tool_parity="${tool_parity}"
+        tool_baud_rate="${tool_baud_rate}"
+        tool_stop_bits="${tool_stop_bits}"
+        tool_rx_idle_chars="${tool_rx_idle_chars}"
+        tool_tx_idle_chars="${tool_tx_idle_chars}"
+        tool_device_name="${tool_device_name}"
+        tool_tcp_port="${tool_tcp_port}"
+        robot_ip="${robot_ip}"
+        script_filename="${script_filename}"
+        output_recipe_filename="${output_recipe_filename}"
+        input_recipe_filename="${input_recipe_filename}"
+        reverse_ip="${reverse_ip}"
+        script_command_port="${script_command_port}"
+        reverse_port="${reverse_port}"
+        script_sender_port="${script_sender_port}"
+        trajectory_port="${trajectory_port}"
     >
-      <origin xyz="0 0.0 0" rpy="0 0 0"/>
+      <origin xyz="0 0 0" rpy="0 0 0"/>
     </xacro:ur_robot>
-    <!-- UR robot -->
-    <!-- <xacro:ur_robot
-      name="${ur_name}"
-      tf_prefix="$(arg tf_prefix)"
-      parent="ur_base_link"
-      joint_limits_parameters_file="$(arg joint_limit_params)"
-      kinematics_parameters_file="$(arg kinematics_params)"
-      physical_parameters_file="$(arg physical_params)"
-      visual_parameters_file="$(arg visual_params)"
-      safety_limits="$(arg safety_limits)"
-      safety_pos_margin="$(arg safety_pos_margin)"
-      safety_k_position="$(arg safety_k_position)"
-      force_abs_paths="$(arg force_abs_paths)"
-      >
-      <origin xyz="0 0 0" rpy="0 0 0" />
-    </xacro:ur_robot> -->
     <!-- Tool holder on tool0 -->
     <xacro:tool_holder parent_link="tool0"/>

Commit message: updating arpa_system with parker linear acutator urdf package

File: src/arpa_description/urdf/arpa_system_macro.urdf.xacro (robot description, xacro)
@@ -8,4 +8,5 @@
   <xacro:include filename="$(find ur_description)/urdf/ur_macro.xacro"/>
   <xacro:include filename="$(find arpa_moveit_config)/config/arpa_system.ros2_control.xacro" />
+  <xacro:include filename="$(find parker_controller_interface)/urdf/parker_linear_actuator_macro.urdf.xacro" />
   <xacro:include filename="$(find parker_controller_interface)/urdf/parker_linear_actuator.ros2_control.xacro" />
   <!-- Macro definition -->
@@ -62,10 +63,10 @@
     </joint>
     <!-- Fixed transform from gantry_link to linear_actuator_link -->
-    <joint name="gantry_to_linear_actuator" type="fixed">
+    <!-- <joint name="gantry_to_linear_actuator" type="fixed">
       <parent link="gantry_link"/>
       <child link="linear_actuator_link"/>
       <origin xyz="0 0 -0.11375" rpy="0 0 0"/>
-    </joint>
-    <xacro:linear_actuator/>
+    </joint> -->
+    <xacro:parker_linear_actuator  attach_link="gantry_link" origin="0 0 -0.11375 0 0 0"/>
     <link name="arm_mount_plate">
       <visual>

File: src/arpa_moveit_config/config/arpa_system.ros2_control.xacro (robot description, xacro)
@@ -1,4 +1,5 @@
 <?xml version="1.0"?>
 <robot xmlns:xacro="http://www.ros.org/wiki/xacro">
+  <xacro:include filename="$(find parker_controller_interface)/urdf/parker_linear_actuator.ros2_control.xacro" />
   <xacro:macro name="arpa_system_ros2_control" params="
     name
@@ -61,4 +62,10 @@
           <param name="tool_tcp_port">${tool_tcp_port}</param>
           <param name="keep_alive_count">${keep_alive_count}</param>
+            <!-- Add ros2_control hardware interface
+          <xacro:parker_linear_actuator_ros2_control
+            name="ParkerControllerInterface"
+            host="192.168.100.1"
+            port="5002"/>
+          </xacro:macro> -->
         </xacro:unless>
       </hardware>

File: src/parker_controller_interface/urdf/parker_linear_actuator_macro.urdf.xacro (robot description, xacro)
@@ -1,4 +1,6 @@
 <?xml version="1.0"?>
-<robot xmlns:xacro="http://www.ros.org/wiki/xacro" name="parker_linear_actuator_robot">
+<robot xmlns:xacro="http://www.ros.org/wiki/xacro" name="parker_linear_actuator_robot" params="
+    attach_link
+    origin">
   <!-- Include ros2_control xacro macros -->
   <xacro:include filename="$(find parker_controller_interface)/urdf/parker_linear_actuator.ros2_control.xacro" />
@@ -24,4 +26,9 @@
       </inertial>
     </link>
+    <joint name="${attach_link}_to_linear_actuator_joint" type="fixed">
+      <parent link="${attach_link}"/>
+      <child link="linear_actuator_link"/>
+      <origin xyz="${origin.split(' ')[0]} ${origin.split(' ')[1]} ${origin.split(' ')[2]}" rpy="${origin.split(' ')[3]} ${origin.split(' ')[4]} ${origin.split(' ')[5]}"/>
+    </joint>
     <link name="linear_actuator_plate_link">
       <visual>

Commit message: WIP: Real arm reintegration - trajectory tolerance fixes and Parker controller updates

File: src/arpa_description/urdf/arpa_system_macro.urdf.xacro (robot description, xacro)
@@ -3,11 +3,10 @@
   <!-- Sub-components -->
   <xacro:include filename="$(find arpa_description)/urdf/gantry.xacro"/>
-  <xacro:include filename="$(find arpa_description)/urdf/linear_actuator.xacro"/>
-  <xacro:include filename="$(find arpa_description)/urdf/linear_actuator_ros2_control.xacro"/>
+  <!-- Linear actuator from parker_controller_interface (0.1-2.0m range, includes visual and ros2_control) -->
+  <xacro:include filename="$(find parker_controller_interface)/urdf/parker_linear_actuator_macro.urdf.xacro" />
+  <xacro:include filename="$(find parker_controller_interface)/urdf/parker_linear_actuator.ros2_control.xacro" />
   <xacro:include filename="$(find arpa_description)/urdf/tool_holder.xacro"/>
   <xacro:include filename="$(find ur_description)/urdf/ur_macro.xacro"/>
   <xacro:include filename="$(find arpa_moveit_config)/config/arpa_system.ros2_control.xacro" />
-  <xacro:include filename="$(find parker_controller_interface)/urdf/parker_linear_actuator_macro.urdf.xacro" />
-  <xacro:include filename="$(find parker_controller_interface)/urdf/parker_linear_actuator.ros2_control.xacro" />
   <!-- Macro definition -->
   <xacro:macro name="arpa_system_macro" params="
@@ -68,5 +67,5 @@
       <origin xyz="0 0 -0.11375" rpy="0 0 0"/>
     </joint> -->
-    <xacro:parker_linear_actuator  attach_link="gantry_link" origin="0 0 -0.11375 0 0 0"/>
+    <xacro:parker_linear_actuator attach_link="gantry_link" origin="0 0 -0.11375 0 0 0"/>
     <link name="arm_mount_plate">
       <visual>

File: src/arpa_description/urdf/linear_actuator.xacro (robot description, xacro)
@@ -48,11 +48,12 @@
       </inertial>
     </link>
-    <!-- Prismatic joint for linear actuator movement -->
+    <!-- Prismatic joint for linear actuator movement (0.1-2.0m = 100-2000mm) -->
+    <!-- NOTE: This macro is deprecated - use parker_linear_actuator from parker_controller_interface instead -->
     <joint name="linear_actuator_to_linear_actuator_plate_joint" type="prismatic">
       <parent link="linear_actuator_link"/>
       <child link="linear_actuator_plate_link"/>
       <origin xyz="1.0244 0 -0.04375" rpy="0 0 0"/>
-      <axis xyz="1 0 0"/>
-      <limit lower="-1.845" upper="0.0" effort="100.0" velocity="0.5"/>
+      <axis xyz="-1 0 0"/>
+      <limit lower="0.1" upper="2.0" effort="100.0" velocity="0.5"/>
     </joint>
   </xacro:macro>

File: src/parker_controller_interface/urdf/parker_linear_actuator.ros2_control.xacro (robot description, xacro)
@@ -17,14 +17,14 @@
           <param name="initial_value">0.0</param>
         </state_interface>
-        <!-- <state_interface name="velocity">
+        <state_interface name="velocity">
           <param name="initial_value">0.0</param>
         </state_interface>
-        <state_interface name="effort">
+        <!-- <state_interface name="effort">
           <param name="initial_value">0.0</param>
         </state_interface> -->
-        <!-- Command interfaces -->
+        <!-- Command interfaces (in meters, 0.1-2.0m = 100-2000mm) -->
         <command_interface name="position">
-          <param name="min">0.0</param>
-          <param name="max">0.5</param>
+          <param name="min">0.1</param>
+          <param name="max">2.0</param>
         </command_interface>
         <!-- <command_interface name="velocity">

File: src/parker_controller_interface/urdf/parker_linear_actuator.urdf.xacro (robot description, xacro)
@@ -14,11 +14,5 @@
     </visual>
   </link>
-  <!-- Fixed joint to attach actuator to world -->
-  <joint name="world_to_actuator_joint" type="fixed">
-    <parent link="world"/>
-    <child link="linear_actuator_link"/>
-    <origin xyz="0 0 0.05" rpy="0 0 0"/>
-  </joint>
   <!-- Instantiate the Parker linear actuator macro -->
-  <xacro:parker_linear_actuator />
+  <xacro:parker_linear_actuator attach_link="world" origin="0 0 0.05 0 0 0"/>
 </robot>

File: src/parker_controller_interface/urdf/parker_linear_actuator_macro.urdf.xacro (robot description, xacro)
@@ -3,7 +3,9 @@
     attach_link
     origin">
+   <xacro:arg name="attach_link" default="" />
+   <xacro:arg name="origin" default="" />
   <!-- Include ros2_control xacro macros -->
   <xacro:include filename="$(find parker_controller_interface)/urdf/parker_linear_actuator.ros2_control.xacro" />
-  <xacro:macro name="parker_linear_actuator">
+  <xacro:macro name="parker_linear_actuator" params="attach_link origin">
     <link name="linear_actuator_link">
       <visual>
@@ -51,11 +53,11 @@
       </inertial>
     </link>
-    <!-- Prismatic joint for linear actuator movement -->
+    <!-- Prismatic joint for linear actuator movement (0.1-2.0m = 100-2000mm) -->
     <joint name="linear_actuator_to_linear_actuator_plate_joint" type="prismatic">
       <parent link="linear_actuator_link"/>
       <child link="linear_actuator_plate_link"/>
       <origin xyz="1.0244 0 -0.04375" rpy="0 0 0"/>
-      <axis xyz="1 0 0"/>
-      <limit lower="-1.845" upper="0.0" effort="100.0" velocity="0.5"/>
+      <axis xyz="-1 0 0"/>
+      <limit lower="0.1" upper="2.0" effort="100.0" velocity="0.5"/>
     </joint>
     <!-- Add ros2_control hardware interface -->
