Commit message: Add gazebo_ros2_control as submodule

File: src/arpa_description/urdf/arpa_system_macro.urdf.xacro (robot description, xacro)
@@ -83,4 +83,32 @@
       <origin xyz="0 0 1.9419" rpy="0 0 0"/>
     </joint>
+    <!-- Battery table at centre of gantry -->
+    <link name="battery_link">
+      <visual>
+        <geometry>
+          <mesh filename="file://$(find arpa_description)/meshes/battery.stl" scale="1.0 1.0 1.0"/>
+        </geometry>
+        <origin xyz="0 0 0" rpy="0 0 0"/>
+        <material name="gantry_gray"/>
+      </visual>
+      <collision>
+        <geometry>
+          <mesh filename="file://$(find arpa_description)/meshes/battery.stl" scale="1.0 1.0 1.0"/>
+        </geometry>
+        <origin xyz="0 0 0" rpy="0 0 0"/>
+      </collision>
+      <inertial>
+        <mass value="10.0"/>
+        <inertia ixx="0.1" ixy="0.0" ixz="0.0"
+                 iyy="0.1" iyz="0.0"
+                 izz="0.1"/>
+      </inertial>
+    </link>
+    <!-- Battery ~50 cm above ground, rotated 90 deg around Z -->
+    <joint name="gantry_to_battery" type="fixed">
+      <parent link="gantry_link"/>
+      <child link="battery_link"/>
+      <origin xyz="0 0 -1.4419" rpy="0 0 1.5708"/>
+    </joint>
     <xacro:linear_actuator/>
     <!-- Fixed transform from gantry_link to linear_actuator_link -->
@@ -168,5 +196,5 @@
     </xacro:ur_robot>
     <!-- Tool holder on tool0 -->
-    <xacro:tool_holder parent_link="tool0"/>
+    <xacro:tool_holder parent_link="tool0" sim_gazebo="${sim_gazebo}"/>
   </xacro:macro>
 </robot>

File: src/arpa_description/urdf/materials.xacro (robot description, xacro)
@@ -11,4 +11,7 @@
       <color rgba="0.6 0.6 0.6 1"/>
     </material>
+    <material name="camera_black">
+      <color rgba="0.1 0.1 0.1 1"/>
+    </material>
   </xacro:macro>
 </robot>

File: src/arpa_description/urdf/tool_holder.xacro (robot description, xacro)
@@ -1,23 +1,36 @@
 <?xml version="1.0"?>
 <robot xmlns:xacro="http://www.ros.org/wiki/xacro">
+  <!-- Materials (pillar_gray, gantry_gray, camera_black, etc.) defined in gantry.xacro via default_materials -->
   <!--
     Macro to attach a tool holder to a parent link (default: tool0)
     Usage:
       <xacro:tool_holder parent_link="tool0"/>
+    How the nut runner gets into the simulation:
+    The runner is part of the single robot URDF (arpa_system.urdf.xacro).
+    Launch runs xacro -> robot_state_publisher gets full description -> spawn_entity
+    spawns the whole robot "ur" into Gazebo. The runner is one link in that tree;
+    there is no separate spawn. Its pose in sim is exactly runner_mount_xyz + runner_mount_rpy
+    (joint block_to_runner_joint). Rebuild arpa_description after changing this file.
   -->
   <xacro:macro name="tool_holder" params="
       parent_link
-      mesh_filename:='$(find arpa_description)/meshes/tool_holder.stl'
+      block_mesh:='$(find arpa_description)/meshes/tool_holder.stl'
+      block_origin_xyz:='-0.0055 -0.0055 -0.006'
+      block_origin_rpy:='${pi/2.} ${3*pi/2.} 0'
+      runner_mesh:='$(find arpa_description)/meshes/realrunner.stl'
+      runner_origin_xyz:='0.0445 -0.0055 -0.006'
+      runner_origin_rpy:='0 0 ${pi}'
+      runner_mount_xyz:='0.08 0 -0.025'
+      runner_mount_rpy:='0 ${pi} ${pi/2.}'
       mass:=0.5
-      origin_xyz:='-0.0055 -0.0055 -.006'
-      origin_rpy:='${pi/2.} ${3*pi/2.} 0'
-      scale:='1.0 1.0 1.0'">
-    <!-- Tool Holder Link -->
+      scale:='1.0 1.0 1.0'
+      sim_gazebo:=false">
+    <!-- Grey block (tool holder) at wrist -->
     <link name="tool_holder_link">
       <visual>
         <geometry>
-          <mesh filename="file://${mesh_filename}" scale="${scale}"/>
-        </geometry>
-        <origin xyz="${origin_xyz}" rpy="${origin_rpy}"/>
+          <mesh filename="file://${block_mesh}" scale="${scale}"/>
+        </geometry>
+        <origin xyz="${block_origin_xyz}" rpy="${block_origin_rpy}"/>
         <material name="grey">
           <color rgba="0.5 0.5 0.5 1.0"/>
@@ -26,7 +39,7 @@
       <collision>
         <geometry>
-          <mesh filename="file://${mesh_filename}" scale="${scale}"/>
-        </geometry>
-        <origin xyz="${origin_xyz}" rpy="${origin_rpy}"/>
+          <mesh filename="file://${block_mesh}" scale="${scale}"/>
+        </geometry>
+        <origin xyz="${block_origin_xyz}" rpy="${block_origin_rpy}"/>
       </collision>
       <inertial>
@@ -38,14 +51,43 @@
       </inertial>
     </link>
-    <!-- Fixed joint to attach to the parent link -->
     <joint name="ur_tool_holder_mount" type="fixed">
       <parent link="${parent_link}"/>
       <child link="tool_holder_link"/>
-      <origin xyz="${origin_xyz}" rpy="${origin_rpy}"/>
-    </joint>
-    <link name="tool_center_link">
-      <visual>
-        <geometry>
-          <cylinder radius=".025" length="0.4"/>
+      <origin xyz="${block_origin_xyz}" rpy="${block_origin_rpy}"/>
+    </joint>
+    <!-- Nut runner tool (below block) -->
+    <link name="runner_link">
+      <visual>
+        <geometry>
+          <mesh filename="file://${runner_mesh}" scale="${scale}"/>
+        </geometry>
+        <origin xyz="${runner_origin_xyz}" rpy="${runner_origin_rpy}"/>
+        <material name="grey">
+          <color rgba="0.5 0.5 0.5 1.0"/>
+        </material>
+      </visual>
+      <collision>
+        <geometry>
+          <mesh filename="file://${runner_mesh}" scale="${scale}"/>
+        </geometry>
+        <origin xyz="${runner_origin_xyz}" rpy="${runner_origin_rpy}"/>
+      </collision>
+      <inertial>
+        <mass value="${mass}"/>
+        <origin xyz="0 0 0" rpy="0 0 0"/>
+        <inertia ixx="0.0001" ixy="0.0" ixz="0.0"
+                 iyy="0.0001" iyz="0.0"
+                 izz="0.0001"/>
+      </inertial>
+    </link>
+    <joint name="block_to_runner_joint" type="fixed">
+      <parent link="tool_holder_link"/>
+      <child link="runner_link"/>
+      <origin xyz="${runner_mount_xyz}" rpy="${runner_mount_rpy}"/>
+    </joint>
+    <link name="tool_head_link">
+      <visual>
+        <geometry>
+          <cylinder radius=".005" length="0.1"/>
         </geometry>
         <origin xyz="0 0 0"/>
@@ -54,5 +96,5 @@
       <collision>
         <geometry>
-          <cylinder radius=".025" length="0.4"/>
+          <cylinder radius=".01" length="0.12"/>
         </geometry>
       </collision>
@@ -62,32 +104,115 @@
       </inertial>
     </link>
-    <joint name="mount_to_center_joint" type="fixed">
-      <parent link="tool_holder_link"/>
-      <child link="tool_center_link"/>
-      <origin xyz="0.0575 0 -0.03" rpy="0 0 0"/>
-    </joint>
-    <link name="tool_head_link">
-      <visual>
-        <geometry>
-          <cylinder radius=".005" length="0.1"/>
-        </geometry>
-        <origin xyz="0 0 0"/>
-        <material name="gantry_gray"/>
-      </visual>
-      <collision>
-        <geometry>
-          <cylinder radius=".01" length="0.12"/>
-        </geometry>
-      </collision>
-      <inertial>
-        <mass value="5.0"/>
-        <inertia ixx="0.01" iyy="0.01" izz="0.01" ixy="0" ixz="0" iyz="0"/>
-      </inertial>
-    </link>
-    <joint name="center_to_tool_head_joint" type="fixed">
-      <parent link="tool_center_link"/>
+    <joint name="runner_to_tool_head_joint" type="fixed">
+      <parent link="runner_link"/>
       <child link="tool_head_link"/>
       <origin xyz="0.06 0 0.175" rpy="0 ${pi/2.} 0"/>
     </joint>
+    <!-- RealSense Camera Link (mounted on tool head) -->
+    <link name="ee_cam_link">
+      <visual>
+        <geometry>
+          <box size="0.025 0.09 0.025"/>
+        </geometry>
+        <origin xyz="0 0 0" rpy="0 0 0"/>
+        <material name="camera_black"/>
+      </visual>
+      <collision>
+        <geometry>
+          <box size="0.025 0.09 0.025"/>
+        </geometry>
+      </collision>
+      <inertial>
+        <mass value="0.1"/>
+        <inertia ixx="0.0001" ixy="0.0" ixz="0.0"
+                 iyy="0.0001" iyz="0.0"
+                 izz="0.0001"/>
+      </inertial>
+    </link>
+    <!-- Camera mount joint (positioned back toward runner to reduce forearm/tool_head collisions) -->
+    <joint name="tool_head_to_camera" type="fixed">
+      <parent link="tool_head_link"/>
+      <child link="ee_cam_link"/>
+      <origin xyz="0 -0.04 0.02" rpy="-1.5708 0 -1.5708"/>
+    </joint>
+    <!-- RGB Camera Optical Frame -->
+    <link name="ee_cam_color_optical_frame"/>
+    <joint name="ee_cam_to_color_optical" type="fixed">
+      <parent link="ee_cam_link"/>
+      <child link="ee_cam_color_optical_frame"/>
+      <origin xyz="0 0 0" rpy="-1.5708 0 -1.5708"/>
+    </joint>
+    <!-- Depth Camera Optical Frame -->
+    <link name="ee_cam_depth_optical_frame"/>
+    <joint name="ee_cam_to_depth_optical" type="fixed">
+      <parent link="ee_cam_link"/>
+      <child link="ee_cam_depth_optical_frame"/>
+      <origin xyz="0 0 0" rpy="-1.5708 0 -1.5708"/>
+    </joint>
+    <!-- Gazebo plugins for camera (only in simulation) -->
+    <xacro:if value="${sim_gazebo}">
+      <!-- RGB Camera Plugin -->
+      <gazebo reference="ee_cam_link">
+        <sensor name="ee_cam_color_sensor" type="camera">
+          <update_rate>30</update_rate>
+          <camera name="ee_cam_color">
+            <horizontal_fov>1.047198</horizontal_fov>  <!-- ~60 degrees -->
+            <image>
+              <width>640</width>
+              <height>480</height>
+              <format>R8G8B8</format>
+            </image>
+            <clip>
+              <near>0.02</near>
+              <far>3.0</far>
+            </clip>
+          </camera>
+          <plugin name="ee_cam_color_plugin" filename="libgazebo_ros_camera.so">
+            <ros>
+              <namespace>/realsense/ee_cam</namespace>
+              <remapping>image_raw:=color/image_raw</remapping>
+              <remapping>image_depth:=depth/image_raw</remapping>
+              <remapping>camera_info:=color/camera_info</remapping>
+              <remapping>camera_info_depth:=depth/camera_info</remapping>
+            </ros>
+            <camera_name>ee_cam</camera_name>
+            <frame_name>ee_cam_color_optical_frame</frame_name>
+            <hack_baseline>0.0</hack_baseline>
+            <min_depth>0.0</min_depth>
+            <max_depth>3.0</max_depth>
+          </plugin>
+        </sensor>
+      </gazebo>
+      <!-- Depth Camera Plugin -->
+      <gazebo reference="ee_cam_link">
+        <sensor name="ee_cam_depth_sensor" type="depth">
+          <update_rate>30</update_rate>
+          <camera name="ee_cam_depth">
+            <horizontal_fov>1.047198</horizontal_fov>  <!-- ~60 degrees -->
+            <image>
+              <width>640</width>
+              <height>480</height>
+              <format>R8G8B8</format>
+            </image>
+            <clip>
+              <near>0.02</near>
+              <far>3.0</far>
+            </clip>
+          </camera>
+          <plugin name="ee_cam_depth_plugin" filename="libgazebo_ros_depth_camera.so">
+            <ros>
+              <namespace>/realsense/ee_cam</namespace>
+              <remapping>image_raw:=depth/image_raw</remapping>
+              <remapping>camera_info:=depth/camera_info</remapping>
+            </ros>
+            <camera_name>ee_cam</camera_name>
+            <frame_name>ee_cam_depth_optical_frame</frame_name>
+            <hack_baseline>0.0</hack_baseline>
+            <min_depth>0.0</min_depth>
+            <max_depth>3.0</max_depth>
+          </plugin>
+        </sensor>
+      </gazebo>
+    </xacro:if>
   </xacro:macro>
 </robot>

File: src/arpa_moveit_config/srdf/arpa_system_macro.srdf.xacro (robot description, xacro)
@@ -75,4 +75,5 @@
     <disable_collisions link1="${prefix}forearm_link" link2="${prefix}upper_arm_link" reason="Adjacent"/>
     <disable_collisions link1="${prefix}forearm_link" link2="${prefix}wrist_1_link" reason="Adjacent"/>
+    <disable_collisions link1="${prefix}forearm_link" link2="${prefix}runner_link" reason="Adjacent"/>
     <disable_collisions link1="${prefix}gantry_link" link2="${prefix}left_leg_link" reason="Never"/>
     <disable_collisions link1="${prefix}gantry_link" link2="${prefix}linear_actuator_link" reason="Adjacent"/>
@@ -88,5 +89,5 @@
     <disable_collisions link1="${prefix}left_leg_link" link2="${prefix}right_leg_link" reason="Never"/>
     <disable_collisions link1="${prefix}left_leg_link" link2="${prefix}shoulder_link" reason="Never"/>
-    <disable_collisions link1="${prefix}left_leg_link" link2="${prefix}tool_center_link" reason="Never"/>
+    <disable_collisions link1="${prefix}left_leg_link" link2="${prefix}runner_link" reason="Never"/>
     <disable_collisions link1="${prefix}left_leg_link" link2="${prefix}tool_head_link" reason="Never"/>
     <disable_collisions link1="${prefix}left_leg_link" link2="${prefix}tool_holder_link" reason="Never"/>
@@ -111,5 +112,5 @@
     <disable_collisions link1="${prefix}pillar_right_link" link2="${prefix}upper_arm_link" reason="Never"/>
     <disable_collisions link1="${prefix}right_leg_link" link2="${prefix}shoulder_link" reason="Never"/>
-    <disable_collisions link1="${prefix}right_leg_link" link2="${prefix}tool_center_link" reason="Never"/>
+    <disable_collisions link1="${prefix}right_leg_link" link2="${prefix}runner_link" reason="Never"/>
     <disable_collisions link1="${prefix}right_leg_link" link2="${prefix}tool_head_link" reason="Never"/>
     <disable_collisions link1="${prefix}right_leg_link" link2="${prefix}tool_holder_link" reason="Never"/>
@@ -120,10 +121,15 @@
     <disable_collisions link1="${prefix}shoulder_link" link2="${prefix}upper_arm_link" reason="Adjacent"/>
     <disable_collisions link1="${prefix}shoulder_link" link2="${prefix}wrist_1_link" reason="Never"/>
-    <disable_collisions link1="${prefix}tool_center_link" link2="${prefix}tool_head_link" reason="Adjacent"/>
-    <disable_collisions link1="${prefix}tool_center_link" link2="${prefix}tool_holder_link" reason="Adjacent"/>
-    <disable_collisions link1="${prefix}tool_center_link" link2="${prefix}wrist_1_link" reason="Never"/>
-    <disable_collisions link1="${prefix}tool_center_link" link2="${prefix}wrist_2_link" reason="Never"/>
-    <disable_collisions link1="${prefix}tool_center_link" link2="${prefix}wrist_3_link" reason="Never"/>
+    <disable_collisions link1="${prefix}runner_link" link2="${prefix}tool_head_link" reason="Adjacent"/>
+    <disable_collisions link1="${prefix}runner_link" link2="${prefix}tool_holder_link" reason="Adjacent"/>
+    <disable_collisions link1="${prefix}runner_link" link2="${prefix}wrist_1_link" reason="Never"/>
+    <disable_collisions link1="${prefix}runner_link" link2="${prefix}wrist_2_link" reason="Never"/>
+    <disable_collisions link1="${prefix}runner_link" link2="${prefix}wrist_3_link" reason="Never"/>
+    <disable_collisions link1="${prefix}ee_cam_link" link2="${prefix}forearm_link" reason="Default"/>
+    <disable_collisions link1="${prefix}ee_cam_link" link2="${prefix}tool_head_link" reason="Adjacent"/>
+    <disable_collisions link1="${prefix}ee_cam_link" link2="${prefix}wrist_1_link" reason="Default"/>
+    <disable_collisions link1="${prefix}battery_link" link2="${prefix}ee_cam_link" reason="Default"/>
     <disable_collisions link1="${prefix}tool_head_link" link2="${prefix}tool_holder_link" reason="Never"/>
+    <disable_collisions link1="${prefix}tool_head_link" link2="${prefix}forearm_link" reason="Default"/>
     <disable_collisions link1="${prefix}tool_head_link" link2="${prefix}wrist_1_link" reason="Never"/>
     <disable_collisions link1="${prefix}tool_head_link" link2="${prefix}wrist_2_link" reason="Never"/>
