Commit message: screw sequence nearly done without cartesian planning

File: src/arpa_description/urdf/arpa_system_macro.urdf.xacro (robot description, xacro)
@@ -6,4 +6,6 @@
   <xacro:include filename="$(find arpa_description)/urdf/linear_actuator_ros2_control.xacro"/>
   <xacro:include filename="$(find arpa_description)/urdf/tool_holder.xacro"/>
+  <xacro:include filename="$(find arpa_description)/urdf/runner.xacro"/>
+  <xacro:include filename="$(find arpa_description)/urdf/camera.xacro"/>
   <xacro:include filename="$(find ur_description)/urdf/ur_macro.xacro"/>
   <!-- <xacro:arg name="tf_prefix" default="" />
@@ -196,5 +198,9 @@
     </xacro:ur_robot>
     <!-- Tool holder on tool0 -->
-    <xacro:tool_holder parent_link="tool0" sim_gazebo="${sim_gazebo}"/>
+    <xacro:tool_holder parent_link="tool0"/>
+    <!-- Nut runner attached to tool holder (flipped to face left) -->
+    <xacro:runner parent_link="tool_holder_link" runner_mount_rpy="0 0 ${pi/2}"/>
+    <!-- RealSense camera attached to tool head -->
+    <xacro:camera parent_link="tool_head_link" sim_gazebo="${sim_gazebo}"/>
   </xacro:macro>
 </robot>

File: src/arpa_description/urdf/tool_holder.xacro (robot description, xacro)
@@ -3,13 +3,7 @@
   <!-- Materials (pillar_gray, gantry_gray, camera_black, etc.) defined in gantry.xacro via default_materials -->
   <!--
-    Macro to attach a tool holder to a parent link (default: tool0)
+    Macro to attach a tool holder and camera to a parent link (default: tool0)
     Usage:
-      <xacro:tool_holder parent_link="tool0"/>
-    How the nut runner gets into the simulation:
-    The runner is part of the single robot URDF (arpa_system.urdf.xacro).
-    Launch runs xacro -> robot_state_publisher gets full description -> spawn_entity
-    spawns the whole robot "ur" into Gazebo. The runner is one link in that tree;
-    there is no separate spawn. Its pose in sim is exactly runner_mount_xyz + runner_mount_rpy
-    (joint block_to_runner_joint). Rebuild arpa_description after changing this file.
+      <xacro:tool_holder parent_link="tool0" sim_gazebo="true"/>
   -->
   <xacro:macro name="tool_holder" params="
@@ -18,9 +12,4 @@
       block_origin_xyz:='-0.0055 -0.0055 -0.006'
       block_origin_rpy:='${pi/2.} ${3*pi/2.} 0'
-      runner_mesh:='$(find arpa_description)/meshes/realrunner.stl'
-      runner_origin_xyz:='0.0445 -0.0055 -0.006'
-      runner_origin_rpy:='0 0 ${pi}'
-      runner_mount_xyz:='0.08 0 -0.025'
-      runner_mount_rpy:='0 ${pi} ${pi/2.}'
       mass:=0.5
       scale:='1.0 1.0 1.0'
@@ -56,163 +45,4 @@
       <origin xyz="${block_origin_xyz}" rpy="${block_origin_rpy}"/>
     </joint>
-    <!-- Nut runner tool (below block) -->
-    <link name="runner_link">
-      <visual>
-        <geometry>
-          <mesh filename="file://${runner_mesh}" scale="${scale}"/>
-        </geometry>
-        <origin xyz="${runner_origin_xyz}" rpy="${runner_origin_rpy}"/>
-        <material name="grey">
-          <color rgba="0.5 0.5 0.5 1.0"/>
-        </material>
-      </visual>
-      <collision>
-        <geometry>
-          <mesh filename="file://${runner_mesh}" scale="${scale}"/>
-        </geometry>
-        <origin xyz="${runner_origin_xyz}" rpy="${runner_origin_rpy}"/>
-      </collision>
-      <inertial>
-        <mass value="${mass}"/>
-        <origin xyz="0 0 0" rpy="0 0 0"/>
-        <inertia ixx="0.0001" ixy="0.0" ixz="0.0"
-                 iyy="0.0001" iyz="0.0"
-                 izz="0.0001"/>
-      </inertial>
-    </link>
-    <joint name="block_to_runner_joint" type="fixed">
-      <parent link="tool_holder_link"/>
-      <child link="runner_link"/>
-      <origin xyz="${runner_mount_xyz}" rpy="${runner_mount_rpy}"/>
-    </joint>
-    <link name="tool_head_link">
-      <visual>
-        <geometry>
-          <cylinder radius=".005" length="0.1"/>
-        </geometry>
-        <origin xyz="0 0 0"/>
-        <material name="gantry_gray"/>
-      </visual>
-      <collision>
-        <geometry>
-          <cylinder radius=".01" length="0.12"/>
-        </geometry>
-      </collision>
-      <inertial>
-        <mass value="5.0"/>
-        <inertia ixx="0.01" iyy="0.01" izz="0.01" ixy="0" ixz="0" iyz="0"/>
-      </inertial>
-    </link>
-    <joint name="runner_to_tool_head_joint" type="fixed">
-      <parent link="runner_link"/>
-      <child link="tool_head_link"/>
-      <origin xyz="0.06 0 0.175" rpy="0 ${pi/2.} 0"/>
-    </joint>
-    <!-- RealSense Camera Link (mounted on tool head) -->
-    <link name="ee_cam_link">
-      <visual>
-        <geometry>
-          <box size="0.025 0.09 0.025"/>
-        </geometry>
-        <origin xyz="0 0 0" rpy="0 0 0"/>
-        <material name="camera_black"/>
-      </visual>
-      <collision>
-        <geometry>
-          <box size="0.025 0.09 0.025"/>
-        </geometry>
-      </collision>
-      <inertial>
-        <mass value="0.1"/>
-        <inertia ixx="0.0001" ixy="0.0" ixz="0.0"
-                 iyy="0.0001" iyz="0.0"
-                 izz="0.0001"/>
-      </inertial>
-    </link>
-    <!-- Camera mount joint (positioned back toward runner to reduce forearm/tool_head collisions) -->
-    <joint name="tool_head_to_camera" type="fixed">
-      <parent link="tool_head_link"/>
-      <child link="ee_cam_link"/>
-      <origin xyz="0 -0.04 0.02" rpy="-1.5708 0 -1.5708"/>
-    </joint>
-    <!-- RGB Camera Optical Frame -->
-    <link name="ee_cam_color_optical_frame"/>
-    <joint name="ee_cam_to_color_optical" type="fixed">
-      <parent link="ee_cam_link"/>
-      <child link="ee_cam_color_optical_frame"/>
-      <origin xyz="0 0 0" rpy="-1.5708 0 -1.5708"/>
-    </joint>
-    <!-- Depth Camera Optical Frame -->
-    <link name="ee_cam_depth_optical_frame"/>
-    <joint name="ee_cam_to_depth_optical" type="fixed">
-      <parent link="ee_cam_link"/>
-      <child link="ee_cam_depth_optical_frame"/>
-      <origin xyz="0 0 0" rpy="-1.5708 0 -1.5708"/>
-    </joint>
-    <!-- Gazebo plugins for camera (only in simulation) -->
-    <xacro:if value="${sim_gazebo}">
-      <!-- RGB Camera Plugin -->
-      <gazebo reference="ee_cam_link">
-        <sensor name="ee_cam_color_sensor" type="camera">
-          <update_rate>30</update_rate>
-          <camera name="ee_cam_color">
-            <horizontal_fov>1.047198</horizontal_fov>  <!-- ~60 degrees -->
-            <image>
-              <width>640</width>
-              <height>480</height>
-              <format>R8G8B8</format>
-            </image>
-            <clip>
-              <near>0.02</near>
-              <far>3.0</far>
-            </clip>
-          </camera>
-          <plugin name="ee_cam_color_plugin" filename="libgazebo_ros_camera.so">
-            <ros>
-              <namespace>/realsense/ee_cam</namespace>
-              <remapping>image_raw:=color/image_raw</remapping>
-              <remapping>image_depth:=depth/image_raw</remapping>
-              <remapping>camera_info:=color/camera_info</remapping>
-              <remapping>camera_info_depth:=depth/camera_info</remapping>
-            </ros>
-            <camera_name>ee_cam</camera_name>
-            <frame_name>ee_cam_color_optical_frame</frame_name>
-            <hack_baseline>0.0</hack_baseline>
-            <min_depth>0.0</min_depth>
-            <max_depth>3.0</max_depth>
-          </plugin>
-        </sensor>
-      </gazebo>
-      <!-- Depth Camera Plugin -->
-      <gazebo reference="ee_cam_link">
-        <sensor name="ee_cam_depth_sensor" type="depth">
-          <update_rate>30</update_rate>
-          <camera name="ee_cam_depth">
-            <horizontal_fov>1.047198</horizontal_fov>  <!-- ~60 degrees -->
-            <image>
-              <width>640</width>
-              <height>480</height>
-              <format>R8G8B8</format>
-            </image>
-            <clip>
-              <near>0.02</near>
-              <far>3.0</far>
-            </clip>
-          </camera>
-          <plugin name="ee_cam_depth_plugin" filename="libgazebo_ros_depth_camera.so">
-            <ros>
-              <namespace>/realsense/ee_cam</namespace>
-              <remapping>image_raw:=depth/image_raw</remapping>
-              <remapping>camera_info:=depth/camera_info</remapping>
-            </ros>
-            <camera_name>ee_cam</camera_name>
-            <frame_name>ee_cam_depth_optical_frame</frame_name>
-            <hack_baseline>0.0</hack_baseline>
-            <min_depth>0.0</min_depth>
-            <max_depth>3.0</max_depth>
-          </plugin>
-        </sensor>
-      </gazebo>
-    </xacro:if>
   </xacro:macro>
 </robot>

File: src/arpa_moveit_config/srdf/arpa_system_macro.srdf.xacro (robot description, xacro)
@@ -135,4 +135,5 @@
     <disable_collisions link1="${prefix}tool_head_link" link2="${prefix}wrist_2_link" reason="Never"/>
     <disable_collisions link1="${prefix}tool_head_link" link2="${prefix}wrist_3_link" reason="Never"/>
+    <disable_collisions link1="${prefix}tool_holder_link" link2="${prefix}forearm_link" reason="Adjacent"/>
     <disable_collisions link1="${prefix}tool_holder_link" link2="${prefix}wrist_1_link" reason="Never"/>
     <disable_collisions link1="${prefix}tool_holder_link" link2="${prefix}wrist_2_link" reason="Never"/>

Commit message: vision looks good, working on moving to vision point

File: src/arpa_description/urdf/arpa_system_macro.urdf.xacro (robot description, xacro)
@@ -189,5 +189,5 @@
     <!-- <xacro:runner parent_link="tool_holder_link" runner_mount_rpy="0 0 ${pi/2}"/> -->
     <!-- RealSense camera attached to tool head -->
-    <!-- <xacro:camera parent_link="tool_head_link" sim_gazebo="${sim_gazebo}"/> -->
+    <!-- <xacro:camera parent_link="ratchet_extension_link" sim_gazebo="${sim_gazebo}"/> -->
     <!-- Gazebo ros2_control plugin - required for controller_manager in simulation -->
     <xacro:if value="${sim_gazebo}">

File: src/arpa_description/urdf/camera.xacro (robot description, xacro)
@@ -2,5 +2,5 @@
 <robot xmlns:xacro="http://www.ros.org/wiki/xacro">
   <!--
-    Macro to attach a RealSense camera to a link (typically tool_head_link).
+    Macro to attach a RealSense camera to a link (typically ratchet_extension_link).
     Creates:
     - ee_cam_link: Camera body link
@@ -10,5 +10,5 @@
     Usage:
       <xacro:include filename="$(find arpa_description)/urdf/camera.xacro"/>
-      <xacro:camera parent_link="tool_head_link" sim_gazebo="true"/>
+      <xacro:camera parent_link="ratchet_extension_link" sim_gazebo="true"/>
   -->
   <xacro:macro name="camera" params="

File: src/arpa_description/urdf/runner.xacro (robot description, xacro)
@@ -6,5 +6,5 @@
     - runner_link: The main runner link with mesh geometry
     - block_to_runner_joint: Joint connecting tool_holder_link to runner_link
-    - tool_head_link: Mounting point for camera/end effector
+    - ratchet_extension_link: Mounting point for camera/end effector
     - runner_to_tool_head_joint: Joint connecting runner to tool head
     Usage:
@@ -53,5 +53,5 @@
     </joint>
     <!-- Tool head link (attachment point for camera and end effector) -->
-    <link name="tool_head_link">
+    <link name="ratchet_extension_link">
       <visual>
         <geometry>
@@ -72,7 +72,7 @@
     </link>
     <!-- Mount tool head to runner -->
-    <joint name="runner_to_tool_head_joint" type="fixed">
+    <joint name="runner_to_ratchet_extension_joint" type="fixed">
       <parent link="runner_link"/>
-      <child link="tool_head_link"/>
+      <child link="ratchet_extension_link"/>
       <origin xyz="0.06 0 0.175" rpy="0 ${pi/2.} 0"/>
     </joint>

File: src/arpa_description/urdf/tool_holder.xacro (robot description, xacro)
@@ -67,5 +67,5 @@
       <origin xyz="0.0575 0 -0.03" rpy="0 0 0"/>
     </joint>
-    <link name="tool_head_link">
+    <link name="ratchet_extension_link">
       <visual>
         <geometry>
@@ -86,10 +86,16 @@
       </inertial>
     </link>
-    <joint name="center_to_tool_head_joint" type="fixed">
+    <joint name="center_to_ratchet_extension_joint" type="fixed">
       <parent link="tool_center_link"/>
-      <child link="tool_head_link"/>
+      <child link="ratchet_extension_link"/>
       <!-- <origin xyz="0.06 0 0.175" rpy="0 ${pi/2.} 0"/> -->
       <origin xyz="0.09 0 0.175" rpy="0 ${pi/2.} 0"/>
     </joint>
+    <link name="tool_head_link"/>
+    <joint name="extension_to_tool_head_joint" type="fixed">
+      <parent link="ratchet_extension_link"/>
+      <child link="tool_head_link"/>
+      <origin xyz="0.0 0 0.09" rpy="0 0 0"/>
+    </joint>
   </xacro:macro>
 </robot>

File: src/arpa_moveit_config/srdf/arpa_system_macro.srdf.xacro (robot description, xacro)
@@ -10,5 +10,5 @@
     </group>
     <group name="${prefix}end_effector">
-      <chain base_link="${prefix}tool0" tip_link="${prefix}tool_head_link"/>
+      <chain base_link="${prefix}tool0" tip_link="${prefix}ratchet_extension_link"/>
     </group>
     <group_state group="ur_manipulator" name="home">
@@ -99,5 +99,5 @@
     <disable_collisions link1="left_leg_link" link2="shoulder_link" reason="Never"/>
     <disable_collisions link1="left_leg_link" link2="tool_center_link" reason="Never"/>
-    <disable_collisions link1="left_leg_link" link2="tool_head_link" reason="Never"/>
+    <disable_collisions link1="left_leg_link" link2="ratchet_extension_link" reason="Never"/>
     <disable_collisions link1="left_leg_link" link2="tool_holder_link" reason="Never"/>
     <disable_collisions link1="left_leg_link" link2="upper_arm_link" reason="Never"/>
@@ -122,5 +122,5 @@
     <disable_collisions link1="right_leg_link" link2="shoulder_link" reason="Never"/>
     <disable_collisions link1="right_leg_link" link2="tool_center_link" reason="Never"/>
-    <disable_collisions link1="right_leg_link" link2="tool_head_link" reason="Never"/>
+    <disable_collisions link1="right_leg_link" link2="ratchet_extension_link" reason="Never"/>
     <disable_collisions link1="right_leg_link" link2="tool_holder_link" reason="Never"/>
     <disable_collisions link1="right_leg_link" link2="upper_arm_link" reason="Never"/>
@@ -130,13 +130,13 @@
     <disable_collisions link1="shoulder_link" link2="upper_arm_link" reason="Adjacent"/>
     <disable_collisions link1="shoulder_link" link2="wrist_1_link" reason="Never"/>
-    <disable_collisions link1="tool_center_link" link2="tool_head_link" reason="Adjacent"/>
+    <disable_collisions link1="tool_center_link" link2="ratchet_extension_link" reason="Adjacent"/>
     <disable_collisions link1="tool_center_link" link2="tool_holder_link" reason="Adjacent"/>
     <disable_collisions link1="tool_center_link" link2="wrist_1_link" reason="Never"/>
     <disable_collisions link1="tool_center_link" link2="wrist_2_link" reason="Never"/>
     <disable_collisions link1="tool_center_link" link2="wrist_3_link" reason="Never"/>
-    <disable_collisions link1="tool_head_link" link2="tool_holder_link" reason="Never"/>
-    <disable_collisions link1="tool_head_link" link2="wrist_1_link" reason="Never"/>
-    <disable_collisions link1="tool_head_link" link2="wrist_2_link" reason="Never"/>
-    <disable_collisions link1="tool_head_link" link2="wrist_3_link" reason="Never"/>
+    <disable_collisions link1="ratchet_extension_link" link2="tool_holder_link" reason="Never"/>
+    <disable_collisions link1="ratchet_extension_link" link2="wrist_1_link" reason="Never"/>
+    <disable_collisions link1="ratchet_extension_link" link2="wrist_2_link" reason="Never"/>
+    <disable_collisions link1="ratchet_extension_link" link2="wrist_3_link" reason="Never"/>
     <disable_collisions link1="tool_holder_link" link2="wrist_1_link" reason="Never"/>
     <disable_collisions link1="tool_holder_link" link2="wrist_2_link" reason="Never"/>

Commit message: save before modifying IK/Orientation constraint

File: src/arpa_description/urdf/arpa_system_macro.urdf.xacro (robot description, xacro)
@@ -89,9 +89,9 @@
         </inertial>
       </link>
-      <!-- Battery ~50 cm above ground, rotated 90 deg around Z -->
+      <!-- Battery ~83 cm above ground, rotated 90 deg around Z -->
       <joint name="gantry_to_battery" type="fixed">
         <parent link="gantry_link"/>
         <child link="battery_link"/>
-        <origin xyz="0 0 -1.4419" rpy="0 0 1.5708"/>
+        <origin xyz="0 0 -1.1119" rpy="0 0 1.5708"/>
       </joint>
       <xacro:linear_actuator/>

File: src/parker_controller_interface/urdf/parker_linear_actuator.ros2_control.xacro (robot description, xacro)
@@ -9,5 +9,5 @@
         <param name="min_position">100.0</param>
         <param name="max_position">2000.0</param>
-        <param name="max_velocity">0.1</param>
+        <param name="max_velocity">0.5</param>
         <param name="max_effort">0.1</param>
       </hardware>

Commit message: normalized costs and ran benchmarks without manipulability

File: src/arpa_description/urdf/arpa_system_macro.urdf.xacro (robot description, xacro)
@@ -89,9 +89,9 @@
         </inertial>
       </link>
-      <!-- Battery ~50 cm above ground, rotated 90 deg around Z -->
+      <!-- Battery ~80 cm above ground, rotated 90 deg around Z -->
       <joint name="gantry_to_battery" type="fixed">
         <parent link="gantry_link"/>
         <child link="battery_link"/>
-        <origin xyz="0 0 -1.4419" rpy="0 0 1.5708"/>
+        <origin xyz="0 0 -1.1419" rpy="0 0 1.5708"/>
       </joint>
       <xacro:linear_actuator/>

Commit message: point cloud done

File: src/arpa_description/urdf/arpa_system_macro.urdf.xacro (robot description, xacro)
@@ -89,9 +89,9 @@
         </inertial>
       </link>
-      <!-- Battery ~83 cm above ground, rotated 90 deg around Z -->
+      <!-- Battery ~73 cm above ground, rotated 90 deg around Z -->
       <joint name="gantry_to_battery" type="fixed">
         <parent link="gantry_link"/>
         <child link="battery_link"/>
-        <origin xyz="0 0 -1.1119" rpy="0 0 1.5708"/>
+        <origin xyz="0 0 -1.2119" rpy="0 0 1.5708"/>
       </joint>
       <xacro:linear_actuator/>

Commit message: everything but core functionality changes

File: src/arpa_description/urdf/arpa_system_macro.urdf.xacro (robot description, xacro)
@@ -73,5 +73,5 @@
             <mesh filename="file://$(find arpa_description)/meshes/battery.stl" scale="1.0 1.0 1.0"/>
           </geometry>
-          <origin xyz="0 0 0" rpy="0 0 0"/>
+          <origin xyz="0.0 0.0 0" rpy="0 0 0"/>
           <material name="gantry_gray"/>
         </visual>
@@ -93,5 +93,5 @@
         <parent link="gantry_link"/>
         <child link="battery_link"/>
-        <origin xyz="0 0 -1.2119" rpy="0 0 1.5708"/>
+        <origin xyz="0.067 -0.0235 -1.2119" rpy="0 0 1.5418"/>
       </joint>
       <xacro:linear_actuator/>
