Commit message: grabbed most of the implementation from arpa_ethernet_motor package

File: src/parker_controller_interface/urdf/parker_linear_actuator.ros2_control.xacro (robot description, xacro)
@@ -1,15 +1,10 @@
 <?xml version="1.0"?>
 <robot xmlns:xacro="http://www.ros.org/wiki/xacro">
-  <xacro:macro name="linear_actuator_ros2_control" params="name use_simulation device_port baud_rate">
+  <xacro:macro name="parker_linear_actuator_ros2_control" params="name host port">
     <ros2_control name="${name}" type="actuator">
       <hardware>
-        <plugin>linear_actuator_hardware/LinearActuatorHardware</plugin>
-        <param name="use_simulation">${use_simulation}</param>
-        <param name="device_port">${device_port}</param>
-        <param name="baud_rate">${baud_rate}</param>
-        <param name="min_position">0.0</param>
-        <param name="max_position">0.5</param>
-        <param name="max_velocity">0.1</param>
-        <param name="max_effort">100.0</param>
+        <plugin>parker_controller_interface/ParkerControllerInterface</plugin>
+        <param name="host">${host}</param>
+        <param name="port">${port}</param>
       </hardware>
       <joint name="linear_actuator_joint">

Commit message: parker interface works?

File: src/parker_controller_interface/urdf/parker_linear_actuator.ros2_control.xacro (robot description, xacro)
@@ -7,16 +7,20 @@
         <param name="host">${host}</param>
         <param name="port">${port}</param>
+        <param name="min_position">100.0</param>
+        <param name="max_position">2000.0</param>
+        <param name="max_velocity">1.0</param>
+        <param name="max_effort">1.0</param>
       </hardware>
-      <joint name="linear_actuator_joint">
+      <joint name="linear_actuator_to_linear_actuator_plate_joint">
         <!-- State interfaces -->
         <state_interface name="position">
           <param name="initial_value">0.0</param>
         </state_interface>
-        <state_interface name="velocity">
+        <!-- <state_interface name="velocity">
           <param name="initial_value">0.0</param>
         </state_interface>
         <state_interface name="effort">
           <param name="initial_value">0.0</param>
-        </state_interface>
+        </state_interface> -->
         <!-- Command interfaces -->
         <command_interface name="position">
@@ -24,5 +28,5 @@
           <param name="max">0.5</param>
         </command_interface>
-        <command_interface name="velocity">
+        <!-- <command_interface name="velocity">
           <param name="min">-0.1</param>
           <param name="max">0.1</param>
@@ -31,5 +35,5 @@
           <param name="min">-100.0</param>
           <param name="max">100.0</param>
-        </command_interface>
+        </command_interface> -->
       </joint>
     </ros2_control>

Commit message: working parker

File: src/parker_controller_interface/urdf/parker_linear_actuator.ros2_control.xacro (robot description, xacro)
@@ -9,6 +9,6 @@
         <param name="min_position">100.0</param>
         <param name="max_position">2000.0</param>
-        <param name="max_velocity">1.0</param>
-        <param name="max_effort">1.0</param>
+        <param name="max_velocity">0.1</param>
+        <param name="max_effort">0.1</param>
       </hardware>
       <joint name="linear_actuator_to_linear_actuator_plate_joint">
@@ -25,11 +25,12 @@
         <!-- Command interfaces (in meters, 0.1-2.0m = 100-2000mm) -->
         <command_interface name="position">
-          <param name="min">0.1</param>
-          <param name="max">2.0</param>
+          <param name="min">0.2</param>
+          <param name="max">1.9</param>
         </command_interface>
-        <!-- <command_interface name="velocity">
+        <command_interface name="velocity">
           <param name="min">-0.1</param>
           <param name="max">0.1</param>
         </command_interface>
+        <!--
         <command_interface name="effort">
           <param name="min">-100.0</param>

File: src/parker_controller_interface/urdf/parker_linear_actuator_macro.urdf.xacro (robot description, xacro)
@@ -59,5 +59,5 @@
       <origin xyz="1.0244 0 -0.04375" rpy="0 0 0"/>
       <axis xyz="-1 0 0"/>
-      <limit lower="0.1" upper="2.0" effort="100.0" velocity="0.5"/>
+      <limit lower="0.2" upper="1.9" effort="100.0" velocity="0.1"/>
     </joint>
     <!-- Add ros2_control hardware interface -->

Commit message: starting benchmark, orientation seems to have a problem

File: src/parker_controller_interface/urdf/parker_linear_actuator.ros2_control.xacro (robot description, xacro)
@@ -9,5 +9,5 @@
         <param name="min_position">100.0</param>
         <param name="max_position">2000.0</param>
-        <param name="max_velocity">0.1</param>
+        <param name="max_velocity">0.3</param>
         <param name="max_effort">0.1</param>
       </hardware>

File: src/parker_controller_interface/urdf/parker_linear_actuator_macro.urdf.xacro (robot description, xacro)
@@ -85,5 +85,5 @@
       <origin xyz="1.0244 0 -0.04375" rpy="0 0 0"/>
       <axis xyz="-1 0 0"/>
-      <limit lower="0.2" upper="1.9" effort="100.0" velocity="0.1"/>
+      <limit lower="0.2" upper="1.9" effort="100.0" velocity="0.3"/>
     </joint>
     <!-- Add ros2_control hardware interface -->
