Commit message: finally controlling with move group instance

File: src/parker_controller_interface/srdf/parker_linear_actuator_macro.srdf.xacro (robot description, xacro)
@@ -6,5 +6,5 @@
     </group>
     <group_state name="actuator_home" group="parker_linear_actuator">
-      <joint name="linear_actuator_to_linear_actuator_plate_joint" value="-1.12"/>
+      <joint name="linear_actuator_to_linear_actuator_plate_joint" value="0.9"/>
     </group_state>
     <virtual_joint name="world" type="fixed" parent_frame="world" child_link="${prefix}floor_link"/>
