Commit message: moving the 'home' linear actuator location to within bounds

File: src/arpa_moveit_config/srdf/arpa_system_macro.srdf.xacro (robot description, xacro)
@@ -31,5 +31,5 @@
     </group>
     <group_state name="actuator_home" group="linear_actuator_axis">
-      <joint name="linear_actuator_to_linear_actuator_plate_joint" value="-1.12"/>
+      <joint name="linear_actuator_to_linear_actuator_plate_joint" value="0.45"/>
     </group_state>
     <group_state name="arm_home" group="ur_manipulator">
@@ -42,5 +42,5 @@
     </group_state>
     <group_state name="arpa_home" group="ur16e_on_gantry">
-      <joint name="linear_actuator_to_linear_actuator_plate_joint" value="-1.12"/>
+      <joint name="linear_actuator_to_linear_actuator_plate_joint" value="0.45"/>
       <joint name="shoulder_pan_joint" value="-2.7576"/>
       <joint name="shoulder_lift_joint" value="-2.6179"/>
